File: hardware/qpcb/kicad/psu.kicad_sch (KiCad schematic)
At the start: 168 parts, among them IC1 LT3083EQ#PBF, IC2 TPS5450QDDARQ1, IC3 LT3083EQ#PBF, IC4 LT3083EQ#PBF, IC5 TPS5450QDDARQ1, IC6 ADM7150ARDZ-3.3-R7, IC7 ADM7150ARDZ-3.3-R7, IC8 ADM7150ARDZ-5.0-R7, IC9 ADM7150ARDZ-5.0-R7, J10 Conn_01x02, J11 Conn_01x02, J12 Conn_01x02, J13 Conn_01x02, J14 Conn_01x02, J15 Conn_01x02, J3 Conn_01x02, J4 Conn_01x02, J5 Conn_01x02, J6 Conn_01x02, J7 Conn_01x02, J8 Conn_01x02, J9 Conn_01x02, Q1 2N7002, Q2 2N7002, Q3 2N7002, Q4 2N7002, Q5 2N7002, Q6 2N7002, U2 MC34063AD, U3 LT337TAT

Commit message: Add footprints and 3d CAD models of components
Parts:
- removed J7: Conn_01x02, symbol Connector_Generic:Conn_01x02
- added C60: 10u, footprints:T491C, symbol Device:C
- added J7: Barrel_Jack_Switch, footprints:694106301002_1, symbol Connector:Barrel_Jack_Switch
- added L6: 330u, footprints:DR1050331R, symbol Device:L
- added SW1: SW_SPDT, footprints:SW_500SSP1S2M2QEA, symbol Switch:SW_SPDT
- C1, C12: footprint (none) -> footprints:CAPC6050X550N
- C10, C13, C15, C3, C5, C9: footprint Capacitor_SMD:C_0805_2012Metric_Pad1.18x1.45mm_HandSolder -> footprints:CAPC3225X230N
- C11, C2, C8: Manufacturer (none) -> KYOCERA AVX; Manufacturer Part Number (none) -> 08053C104JAZ2A; Mouser Part Number (none) -> 581-08053C104JAZ2A; Mouser Price/Stock (none) -> https://www.mouser.it/ProductDetail/KYOCERA-AVX/08053C104JA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; Package (none) -> 0805
- C14, C18, C19, C20, C21, C23, C24, C25, C26, C29, C30, C32, C33, C34, C35, C36, C37, C4, C40, C41, C42, C43, R15, R16, R17, R18, R23, R24, R26, R27, R30, R33, R34, R4, R40, R41, R5, R6, R7: footprint (none) -> Capacitor_SMD:C_0805_2012Metric_Pad1.18x1.45mm_HandSolder
- C16, C17: footprint Capacitor_SMD:C_0805_2012Metric_Pad1.18x1.45mm_HandSolder -> footprints:CAPPM3528X210N
- C22, C7: footprint (none) -> footprints:T491C
- C27: footprint Capacitor_SMD:C_0805_2012Metric_Pad1.18x1.45mm_HandSolder -> footprints:CAPC3225X280N; Manufacturer (none) -> TAIYO YUDEN; Manufacturer Part Number (none) -> LMK325ABJ107MM-T; Mouser Part Number (none) -> 963-LMK325ABJ107MM-T; Mouser Price/Stock (none) -> https://www.mouser.it/ProductDetail/TAIYO-YUDEN/LMK325ABJ10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; Package (none) -> 1210
- C28: footprint Capacitor_SMD:C_0805_2012Metric_Pad1.18x1.45mm_HandSolder -> footprints:T521D; Manufacturer (none) -> KEMET; Manufacturer Part Number (none) -> T521D565M050ATE070; Mouser Part Number (none) -> 80-T521D565M50ATE70; Mouser Price/Stock (none) -> https://www.mouser.it/ProductDetail/KEMET/T521D565M050ATE07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; Package (none) -> D Case
- C31: value 190p -> 200p; Manufacturer Part Number 700A191JCA150XC100 -> 600F201JT250XT; Mouser Part Number 581-700A191JCA150100 -> 581-600F201JT; Mouser Price/Stock https://www.mouser.it/ProductDetail/KYOCERA-AVX/700A191JCA1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 -> https://www.mouser.it/ProductDetail/KYOCERA-AVX/600F201JT25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; Package 0505 -> 0805
- C38: footprint Capacitor_SMD:C_0805_2012Metric_Pad1.18x1.45mm_HandSolder -> footprints:CAPPM2014X170N
- C39: footprint Capacitor_SMD:C_0805_2012Metric_Pad1.18x1.45mm_HandSolder -> footprints:EEEFK0J332AV; Manufacturer Nichicon -> Panasonic; Manufacturer Part Number UCZ1J751MNS1MS -> EEE-FK1V751SV; Mouser Part Number 647-UCZ1J751MNS1MS -> 667-EEE-FK1V751SV; Mouser Price/Stock https://www.mouser.it/ProductDetail/Nichicon/UCZ1J751MNS1MS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 -> https://www.mouser.it/ProductDetail/Panasonic/EEE-FK1V751SV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
- C6: footprint Capacitor_SMD:C_0805_2012Metric_Pad1.18x1.45mm_HandSolder -> footprints:16SVF270M; Manufacturer (none) -> Panasonic; Manufacturer Part Number (none) -> 10SVP150MX; Mouser Part Number (none) -> 667-10SVP150MX; Mouser Price/Stock (none) -> https://www.mouser.it/ProductDetail/Panasonic/10SVP150MX?qs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
- D1, D11, D12, D13, D2, D5, D7, D8: footprint (none) -> LED_SMD:LED_0805_2012Metric_Pad1.15x1.40mm_HandSolder
- D10, D16, D17, D3, D4, D9: footprint footprints:SODFL3616X98N -> footprints:RBE01VYM6AFHTR
- D14, D15, D20, D22, D23: footprint (none) -> footprints:PMEG3050EP115
- D18: footprint (none) -> footprints:SODFL3617X108N
- D19: footprint Diode_SMD:D_SOD-128 -> footprints:PMEG3050EP115
- D21: footprint Diode_THT:D_DO-41_SOD81_P10.16mm_Horizontal -> footprints:SOD3716X145N
- D6: footprint (none) -> footprints:SBR10200CTL13
- J10, J11, J12, J13, J14, J15, J3, J4, J5, J6, J8, J9: footprint (none) -> footprints:09652028; Manufacturer (none) -> Molex; Manufacturer Part Number (none) -> 09-65-2028; Mating Crimp (none) -> 538-08-70-1031-CT; Mating Part (none) -> 538-09-50-1021; Mouser Part Number (none) -> 538-09-65-2028; Mouser Price/Stock (none) -> https://www.mouser.it/ProductDetail/Molex/09-65-2028?qs=cRU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
- L1: value 15u -> 22u; footprint (none) -> footprints:IND_SER1390_COC; Manufacturer Part Number MSS1210-153MED -> SER1390-223MLD; Mouser Part Number 994-MSS1210-153MED -> 994-SER1390-223MLD; Mouser Price/Stock https://www.mouser.it/ProductDetail/Coilcraft/MSS1210-153ME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 -> https://www.mouser.it/ProductDetail/Coilcraft/SER1390-223ML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; Package 4747 (1212 metric) -> (none)
- L2, L4: footprint (none) -> footprints:SRP1038WA100M
- L5: footprint (none) -> footprints:ETQ-P4M_KFM; Manufacturer Part Number ETQ-P5M101YGM -> ETQ-P5M101YGM; Mouser Part Number 667-ETQ-P5M101YGM -> 667-ETQ-P5M101YGM
- Q1, Q2, Q3, Q4, Q5, Q6: footprint Package_TO_SOT_SMD:SOT-23 -> footprints:SOT96P240X120-3N
- R1, R19: footprint (none) -> Capacitor_SMD:C_0805_2012Metric_Pad1.18x1.45mm_HandSolder; Manufacturer (none) -> Panasonic; Manufacturer Part Number (none) -> ERA-6AED124V; Mouser Part Number (none) -> 667-ERA-6AED124V; Mouser Price/Stock (none) -> https://www.mouser.it/ProductDetail/Panasonic/ERA-6AED124V?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; Package (none) -> 0805
- R10, R28, R36, R37: footprint (none) -> Capacitor_SMD:C_0805_2012Metric_Pad1.18x1.45mm_HandSolder; Package (none) -> 0805
- R11: footprint (none) -> Capacitor_SMD:C_0805_2012Metric_Pad1.18x1.45mm_HandSolder; Manufacturer (none) -> Vishay; Manufacturer Part Number (none) -> CRCW08051K80FKEA; Mouser Part Number (none) -> 71-CRCW0805-1.8K-E3; Mouser Price/Stock (none) -> https://www.mouser.it/ProductDetail/Vishay-Dale/CRCW08051K8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; Package (none) -> 0805
- R12, R25: value 6k -> 5.9k; footprint (none) -> Capacitor_SMD:C_0805_2012Metric_Pad1.18x1.45mm_HandSolder; Manufacturer (none) -> Vishay; Manufacturer Part Number (none) -> CRCW08055K90FKEA; Mouser Part Number (none) -> 71-CRCW0805-5.9K-E3; Mouser Price/Stock (none) -> https://www.mouser.it/ProductDetail/Vishay-Dale/CRCW08055K9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; Package (none) -> 0805
- R13, R9: value R -> 150; footprint (none) -> Capacitor_SMD:C_0805_2012Metric_Pad1.18x1.45mm_HandSolder; Package (none) -> 0805
- R14, R21, R22: value R -> 68; footprint (none) -> Capacitor_SMD:C_0805_2012Metric_Pad1.18x1.45mm_HandSolder; Package (none) -> 0805
- R2: value R -> 1.1k; footprint (none) -> Capacitor_SMD:C_0805_2012Metric_Pad1.18x1.45mm_HandSolder; Manufacturer (none) -> Panasonic; Manufacturer Part Number (none) -> ERJ-UP6D1101V; Mouser Part Number (none) -> 667-ERJ-UP6D1101V; Mouser Price/Stock (none) -> https://www.mouser.it/ProductDetail/Panasonic/ERJ-UP6D1101V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; Package (none) -> 0805
- R20: value TBD -> 787; footprint (none) -> Capacitor_SMD:C_0805_2012Metric_Pad1.18x1.45mm_HandSolder; Manufacturer (none) -> Vishay; Manufacturer Part Number (none) -> CRCW0805787RFKEA; Mouser Part Number (none) -> 71-CRCW0805-787-E3; Mouser Price/Stock (none) -> https://www.mouser.it/ProductDetail/Vishay-Dale/CRCW0805787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; Package (none) -> 0805
- R29: footprint (none) -> Capacitor_SMD:C_0805_2012Metric_Pad1.18x1.45mm_HandSolder; Manufacturer (none) -> YAGEO; Manufacturer Part Number (none) -> AF0805FR-0712KL; Mouser Part Number (none) -> 603-AF0805FR-0712KL; Mouser Price/Stock (none) -> https://www.mouser.it/ProductDetail/YAGEO/AF0805FR-0712KL?q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; Package (none) -> 0805
- R3: value R -> 510; footprint (none) -> Capacitor_SMD:C_0805_2012Metric_Pad1.18x1.45mm_HandSolder; Manufacturer (none) -> Panasonic; Manufacturer Part Number (none) -> ERJ-UP6D5100V; Mouser Part Number (none) -> 667-ERJ-UP6D5100V; Mouser Price/Stock (none) -> https://www.mouser.it/ProductDetail/Panasonic/ERJ-UP6D5100V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; Package (none) -> 0805
- R31: footprint (none) -> https://www.mouser.it/ProductDetail/Vishay-Dale/CRCW0805953RFKEA?qs=sGAEpiMZZMtlubZbdhIBIP55dmWdEGuB3ZlBKXDeB7I%3D; Package (none) -> 0805
- R32: value TBD -> 1.4k; footprint (none) -> Capacitor_SMD:C_0805_2012Metric_Pad1.18x1.45mm_HandSolder; Manufacturer (none) -> KOA Speer; Manufacturer Part Number (none) -> RK73H2ATTDD1401F; Mouser Part Number (none) -> 660-RK73H2ATTDD1401F; Mouser Price/Stock (none) -> https://www.mouser.it/ProductDetail/KOA-Speer/RK73H2ATTDD14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; Package (none) -> 0805
- R35: footprint (none) -> Resistor_SMD:R_2512_6332Metric_Pad1.40x3.35mm_HandSolder
- R38: value 198 -> 300; footprint (none) -> Capacitor_SMD:C_0805_2012Metric_Pad1.18x1.45mm_HandSolder; Manufacturer (none) -> Panasonic; Manufacturer Part Number (none) -> ERJ-UP6D3000V; Mouser Part Number (none) -> 667-ERJ-UP6D3000V; Mouser Price/Stock (none) -> https://www.mouser.it/ProductDetail/Panasonic/ERJ-UP6D3000V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; Package (none) -> 0805
- R39: value 121 -> 86.6; footprint (none) -> Capacitor_SMD:C_0805_2012Metric_Pad1.18x1.45mm_HandSolder; Manufacturer (none) -> Panasonic; Manufacturer Part Number (none) -> ERA-6AEB86R6V; Mouser Part Number (none) -> 667-ERA-6AEB86R6V; Mouser Price/Stock (none) -> https://www.mouser.it/ProductDetail/Panasonic/ERA-6AEB86R6V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; Package (none) -> 0805
- R8: value R -> 220; footprint (none) -> Capacitor_SMD:C_0805_2012Metric_Pad1.18x1.45mm_HandSolder; Package (none) -> 0805
- U2: footprint Package_SO:SOIC-8_3.9x4.9mm_P1.27mm -> footprints:SOIC127P599X175-8N
- U3: footprint LM337T:TO254P1054X470X1955-3 -> Package_TO_SOT_THT:TO-220-3_Horizontal_TabDown
Connections:
- net -6V_INT: now also C60.2, L6.2; no longer C31.2, C39.2, D21.2 (A), R36.1, U2.4 (GND)
- net 24V: now also SW1.3 (C)
- net GND: now also C60.1, J7.2, J7.3
- new net: C31.2, C39.2, D21.2 (A), L6.1, R36.1, U2.4 (GND)
- new net: J7.1, SW1.2 (B)
- no-connect marks 0 -> 1
Other:
- note added: "The TPS5450-Q1 circuit was designed using TI WEBENCH POWER DESIGNER. The design can be obtained at the following link: https://webench.ti.com/appinfo/webench/scripts/SDP.cgi?ID=D236DE5285518499"
- note removed: "The TPS5450-Q1 circuit was designed using TI WEBENCH POWER DESIGNER. The design can be obtained at the following link: https://webench.ti.com/appinfo/webench/scripts/SDP.cgi?ID=2D7513C0D29458C6"

Commit message: Add final footprints of daughter boards, change components for -3v3 power supply line and placement almost finished
Parts:
- removed U3: LT337TAT, Package_TO_SOT_THT:TO-220-3_Horizontal_TabDown, symbol LM337T:LM337T
- added C13, C14, C16, C17, C2, C21, C24, C25, C26, C36, C41, C42, C43, C44, C48, C49, C5, C58, C62, C65, C66, C8: 0.1u, Capacitor_SMD:C_0805_2012Metric_Pad1.18x1.45mm_HandSolder, symbol Device:C_Small
- added D24: RBE01VYM6AFHTR, footprints:RBE01VYM6AFHTR, symbol MBR120VLSFT1G:MBR120VLSFT1G
- added IC13: LM2991S_NOPB, footprints:TO170P1435X465-6N, symbol LM2991S_NOPB:LM2991S_NOPB
- added JP7: Jumper_2_Open, Connector_PinHeader_2.54mm:PinHeader_1x02_P2.54mm_Vertical, symbol Jumper:Jumper_2_Open
- added Q9: 2N7002, footprints:SOT96P240X120-3N, symbol Transistor_FET:2N7002
- added R74, R75, R76: 100k, Capacitor_SMD:C_0805_2012Metric_Pad1.18x1.45mm_HandSolder, symbol Device:R
- C1: renamed from C2; symbol Device:C_Polarized_US -> Device:C_Small
- C57: renamed from C39; value 750u -> 33u; footprint footprints:EEEFK0J332AV -> footprints:C4532_Commercial; symbol Device:C_Polarized_US -> Device:C; Manufacturer Panasonic -> TDK; Manufacturer Part Number EEE-FK1V751SV -> C4532X5R1C336M250KA; Mouser Part Number 667-EEE-FK1V751SV -> 810-C4532X5R1C336M; Mouser Price/Stock https://www.mouser.it/ProductDetail/Panasonic/EEE-FK1V751SV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 -> https://www.mouser.it/ProductDetail/TDK/C4532X5R1C336M250KA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; Package (none) -> 1812
- JP1, JP2, JP3, JP4, JP5, JP6: footprint (none) -> Connector_PinHeader_2.54mm:PinHeader_1x02_P2.54mm_Vertical
- L3: footprint (none) -> footprints:IHLP3232DZER330M11; Manufacturer (none) -> Vishay; Manufacturer Part Number (none) -> IHLP3232DZER330M11; Mouser Part Number (none) -> 70-IHLP3232DZER330M1; Mouser Price/Stock (none) -> https://www.mouser.it/ProductDetail/Vishay-Dale/IHLP3232DZE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
- R30: renamed from R31; footprint https://www.mouser.it/ProductDetail/Vishay-Dale/CRCW0805953RFKEA?qs=sGAEpiMZZMtlubZbdhIBIP55dmWdEGuB3ZlBKXDeB7I%3D -> Capacitor_SMD:C_0805_2012Metric_Pad1.18x1.45mm_HandSolder
- R38: value 300 -> 576; footprint Capacitor_SMD:C_0805_2012Metric_Pad1.18x1.45mm_HandSolder -> Resistor_SMD:R_0805_2012Metric_Pad1.20x1.40mm_HandSolder; Manufacturer Panasonic -> Vishay; Manufacturer Part Number ERJ-UP6D3000V -> CRCW0805576RFKTA; Mouser Part Number 667-ERJ-UP6D3000V -> 71-CRCW0805-576; Mouser Price/Stock https://www.mouser.it/ProductDetail/Panasonic/ERJ-UP6D3000V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 -> https://www.mouser.it/ProductDetail/Vishay-Dale/CRCW0805576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
- R39: value 86.6 -> 1k
- TP1, TP18, TP19, TP2, TP20: footprint (none) -> TestPoint:TestPoint_Pad_D1.0mm
- TP10: renamed from TP7; footprint (none) -> TestPoint:TestPoint_Pad_D1.0mm
- TP11: renamed from TP8; footprint (none) -> TestPoint:TestPoint_Pad_D1.0mm
- TP12: renamed from TP16; footprint (none) -> TestPoint:TestPoint_Pad_D1.0mm
- TP13: renamed from TP9; footprint (none) -> TestPoint:TestPoint_Pad_D1.0mm
- TP14: renamed from TP10; footprint (none) -> TestPoint:TestPoint_Pad_D1.0mm
- TP15: renamed from TP17; footprint (none) -> TestPoint:TestPoint_Pad_D1.0mm
- TP16: renamed from TP11; footprint (none) -> TestPoint:TestPoint_Pad_D1.0mm
- TP17: renamed from TP12; footprint (none) -> TestPoint:TestPoint_Pad_D1.0mm
- TP3: renamed from TP13; footprint (none) -> TestPoint:TestPoint_Pad_D1.0mm
- TP4: renamed from TP3; footprint (none) -> TestPoint:TestPoint_Pad_D1.0mm
- TP5: renamed from TP4; footprint (none) -> TestPoint:TestPoint_Pad_D1.0mm
- TP6: renamed from TP14; footprint (none) -> TestPoint:TestPoint_Pad_D1.0mm
- TP7: renamed from TP5; footprint (none) -> TestPoint:TestPoint_Pad_D1.0mm
- TP8: renamed from TP6; footprint (none) -> TestPoint:TestPoint_Pad_D1.0mm
- TP9: renamed from TP15; footprint (none) -> TestPoint:TestPoint_Pad_D1.0mm
- renumbered C6 to C10, C9 to C11, C7 to C12, C10 to C15, C11 to C18, C12 to C19, C13 to C20, C14 to C22, C15 to C23, C18 to C27, C19 to C28, C20 to C29, C21 to C30, C16 to C31, C23 to C32, C24 to C33, C17 to C34, C22 to C35, C25 to C37, C26 to C38, C29 to C39, C1 to C4, C30 to C40, C27 to C45, C28 to C46, C31 to C47, C32 to C50, C33 to C51, C34 to C52, C35 to C53, C36 to C54, C37 to C55, C38 to C56, C60 to C59, C5 to C6, C40 to C60, C41 to C61, C42 to C63, C43 to C64, C4 to C7, C8 to C9, D16 to D14, D17 to D15, D14 to D16, D15 to D17, D7 to D6, D8 to D7, D6 to D8, J11 to J10, J12 to J11, J13 to J12, J14 to J13, J15 to J14, J7 to J15, J8 to J7, J9 to J8, J10 to J9, R13 to R10, R12 to R11, R10 to R12, R11 to R13, R21 to R20, R22 to R21, R20 to R22, R26 to R25, R27 to R26, R25 to R27, R30 to R29, R29 to R31
Connections:
- net -3V3: now also C58.1, IC13.5 (OUTPUT)
- net -6V: now also C44.1, IC13.3 (INPUT), IC13.6 (INPUT_1)
- net -6V_INT: now also C62.1
- net 12V: now also C24.1
- net 14V: now also C21.1
- net 14V_INT: now also C36.1
- net 24V: now also C17.1, C2.1
- net 3V3_A: now also C25.1
- net 3V3_B: now also C26.1
- net 3V3_RASP: now also JP7.1 (A), R76.1
- net 5V_A: now also C49.1
- net 5V_B: now also C48.1
- net 6V: now also C8.1
- net 6V_AUX: now also C16.1, C41.1, C42.1
- net 8V: now also C13.1, C43.1, C5.1, C65.1, C66.1
- net 8V_INT: now also C14.1
- net GND: now also C13.2, C14.2, C16.2, C17.2, C2.2, C21.2, C24.2, C25.2, C26.2, C36.2, C41.2, C42.2, C43.2, C44.2, C48.2, C49.2, C5.2, C58.2, C62.2, C65.2, C66.2, C8.2, IC13.4 (GROUND), Q9.2 (S), R74.2
- net at C10.1, L2.1, R12.2: now also L1.2; no longer L1.1
- net at C7.2, D8.1 (K), IC2.8 (PH): now also L1.1; no longer L1.2
- net at R38.2, R39.1: now also IC13.1 (ADJUST)
- new net: D24.1 (K), JP7.2 (B), R74.1, R75.1
- new net: Q9.1 (G), R75.2
- new net -3V3_EN_SW: D24.2 (A)
- new net -3V3_EN_n: IC13.2 (~{ON}/OFF), Q9.3 (D), R76.2
Other:
- moved on the sheet: C10, C12, C27, C28, C29, C30, C32, C33, C37, C38, C39, C4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

Commit message: Add QPCB JLCPCB production files
Parts:
- removed D10, D14, D15, D24, D3, D4, D9: RBE01VYM6AFHTR, footprints:RBE01VYM6AFHTR, symbol MBR120VLSFT1G:MBR120VLSFT1G
- removed JP5, JP6, JP7: Jumper_2_Open, Connector_PinHeader_2.54mm:PinHeader_1x02_P2.54mm_Vertical, symbol Jumper:Jumper_2_Open
- removed Q1, Q2, Q3, Q4, Q5, Q6, Q9: 2N7002, footprints:SOT96P240X120-3N, symbol Transistor_FET:2N7002
- removed R15, R16, R17, R18, R23, R24, R25, R26, R4, R5, R6, R7, R74, R75, R76: 100k, Capacitor_SMD:C_0805_2012Metric_Pad1.18x1.45mm_HandSolder, symbol Device:R
- added JP8, JP9: Jumper_2_Open, Connector_PinHeader_2.54mm:PinHeader_1x02_P2.54mm_Vertical, symbol Jumper:Jumper_2_Open
- C1, C13, C14, C16, C18, C21, C24, C25, C26, C36, C41, C42, C43, C44, C48, C49, C5, C58, C62, C65, C66, C8, C9: LCSC (none) -> C2170167
- C10: LCSC (none) -> C347568
- C11, C15, C20, C23, C3, C6: LCSC (none) -> C2171868
- C12, C35, C59: LCSC (none) -> C1953415
- C17, C2: LCSC (none) -> C18212337
- C19, C4: LCSC (none) -> C2168425
- C22, C7: LCSC (none) -> C128911
- C31, C34: LCSC (none) -> C308917
- C45: LCSC (none) -> C2880380
- C46: LCSC (none) -> C19940639
- C47: LCSC (none) -> C3905935
- C56: LCSC (none) -> C118763
- C57: LCSC (none) -> C2173074
- D1, D11, D12, D13, D2, D5, D6, D7: LCSC (none) -> C5342088
- D16, D17, D19, D20, D22, D23: LCSC (none) -> C50603
- D18: LCSC (none) -> C894433
- D21: LCSC (none) -> C460770
- D8: LCSC (none) -> C459529
- IC1, IC3, IC4: LCSC (none) -> C459910; Manufacturer Part Number (none) -> LT3083EQ#PBF
- IC13: LCSC (none) -> C205474; Manufacturer Part Number (none) -> LM2991S/NOPB
- IC2, IC5: LCSC (none) -> C181270
- IC6, IC7: LCSC (none) -> C658444
- IC8, IC9: LCSC (none) -> C208034
- J10, J11, J12, J13, J14, J3, J4, J5, J6, J7, J8, J9: LCSC (none) -> C239393
- L1: LCSC (none) -> C3911669
- L2, L4: LCSC (none) -> C17496174
- L3: LCSC (none) -> C845055
- L5: LCSC (none) -> C409631
- L6: LCSC (none) -> C2454092
- R1, R19: LCSC (none) -> C2092728
- R11, R27: LCSC (none) -> C2077391
- R13: LCSC (none) -> C844606
- R2: LCSC (none) -> C5687974
- R22: LCSC (none) -> C2080791
- R28: LCSC (none) -> C4071803
- R3: LCSC (none) -> C5635009
- R30: LCSC (none) -> C3009264
- R31: LCSC (none) -> C4092271
- R35: LCSC (none) -> C20520788
- R36: LCSC (none) -> C2089740
- R37: LCSC (none) -> C2080030
- R38: LCSC (none) -> C4337977
- R39: LCSC (none) -> C4118653
- SW1: LCSC (none) -> C6689030
- U2: LCSC (none) -> C236257
Connections:
- net -3V3_EN_n is gone; now on net GND: IC13.2 (~{ON}/OFF)
- net 12V_EN: now also JP4.1 (A)
- net 3V3_A_EN: now also JP8.1 (A)
- net 3V3_B_EN: now also JP9.1 (A)
- net 5V_A_EN: now also JP1.1 (A)
- net 5V_B_EN: now also JP3.1 (A)
- net 6V_EN: now also JP2.1 (A)
- net GND: now also JP1.2 (B), JP2.2 (B), JP3.2 (B), JP4.2 (B), JP8.2 (B), JP9.2 (B)
- removed net 3V3_RASP: JP1.1 (A), JP2.1 (A), JP3.1 (A), JP4.1 (A)
Other:
- note added: "Power-supplies enable jumpers"
- note added: "The input 8V is first converted to -6V using the MC34063AD buck-boost converter. Then, it is regulated at -3.3V using the LM2991 linear voltage regulator. -6V input voltage is required to guarantee the minimum voltage dropout."
- note removed: "Power-supplies enable circuit"
- note removed: "The input 7.5V is first converted to -3.3V using the MC34063AD buck-boost converter. Then, it is regulated at -3.3V using the LT337 linear voltage regulator. 7.5V input voltage is required to guarantee the minimum voltage dropout."
- moved on the sheet: C25, C26, C27, C28, C29, C30, C32, C33, C37, C38, C39, C40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
