File: hardware/qpcb/kicad/qpcb.kicad_pcb (KiCad board)
At the start: 2 copper layers, 280 x 205 mm, 284 parts, among them IC1 LT3083EQ#PBF, IC10 DAC8562TDGSR, IC11 DAC8562TDGSR, IC12 DAC8562TDGSR, IC13 LM2991S_NOPB, IC2 TPS5450QDDARQ1, IC3 LT3083EQ#PBF, IC4 LT3083EQ#PBF, IC5 TPS5450QDDARQ1, IC6 ADM7150ARDZ-3.3-R7, IC7 ADM7150ARDZ-3.3-R7, IC8 ADM7150ARDZ-5.0-R7, IC9 ADM7150ARDZ-5.0-R7, J10 Conn_01x02, J11 Conn_01x02, J12 Conn_01x02, J13 Conn_01x02, J14 Conn_01x02, J15 Barrel_Jack_Switch, J16 Conn_01x04, J17 Conn_01x04, J2 UART0 Connector, J3 Conn_01x02, J4 Conn_01x02, J5 Conn_01x02, J6 Conn_01x02, J7 Conn_01x02, J8 Conn_01x02, J9 Conn_01x02, Q1 2N7002, Q2 2N7002, Q3 2N7002, Q4 2N7002, Q5 2N7002, Q6 2N7002, Q7 NPN, Q8 NPN, Q9 2N7002, SW1 SW_SPDT, U1 Pico, U17 LT1632CS8#PBF, U18 LT1632CS8#PBF, U2 MC34063AD, U21 LT1632CS8#PBF, U22 LT1632CS8#PBF, Y1 SiT5157AI-FK-33N0-100.000000X

Commit message: Add QPCB JLCPCB production files
Parts:
- removed D10, D14, D15, D24, D3, D4, D9: RBE01VYM6AFHTR, footprints:RBE01VYM6AFHTR
- removed JP5, JP6, JP7: Jumper_2_Open, Connector_PinHeader_2.54mm:PinHeader_1x02_P2.54mm_Vertical
- removed Q1, Q2, Q3, Q4, Q5, Q6, Q9: 2N7002, footprints:SOT96P240X120-3N
- removed R15, R16, R17, R18, R23, R24, R25, R26, R4, R5, R6, R7, R74, R75, R76: 100k, Capacitor_SMD:C_0805_2012Metric_Pad1.18x1.45mm_HandSolder
- added JP8: Jumper_2_Open, Connector_PinHeader_2.54mm:PinHeader_1x02_P2.54mm_Vertical, F.Cu at (305.8, 118.9)
- added JP9: Jumper_2_Open, Connector_PinHeader_2.54mm:PinHeader_1x02_P2.54mm_Vertical, F.Cu at (294.9, 181.2)
- C69: moved to F.Cu
- C79, C80, C81, C82, IC12, Q7, Q8, R66, R67, R68, R69, R70, R71, R72, R73, U21, U22: moved to B.Cu
- moved Q8 521.0 mm to (104.8, 211.1), turned to -90 degrees
- moved Q7 517.0 mm to (104.8, 191.1), turned to -90 degrees
- moved U22 510.8 mm to (119.8, 211.1), turned to -90 degrees
- moved R73 509.1 mm to (110.7, 212.5), turned to 180 degrees
- moved U21 506.8 mm to (119.8, 191.1), turned to -90 degrees
- moved R68 504.9 mm to (110.7, 190.0), turned to 180 degrees
- moved R69 504.8 mm to (110.7, 192.5), turned to 180 degrees
- moved C82 499.7 mm to (124.2, 209.7), turned to 90 degrees
- moved C79 496.5 mm to (124.2, 189.7), turned to 90 degrees
- moved R72 495.2 mm to (110.7, 210.0), turned to 180 degrees
- moved R66 495.1 mm to (121.4, 186.2), turned to 180 degrees
- moved R67 493.7 mm to (121.4, 183.7)
- moved C81 489.5 mm to (135.0, 207.3)
- moved C80 487.8 mm to (136.5, 203.3), turned to 90 degrees
- moved R70 485.5 mm to (121.4, 206.2), turned to 180 degrees
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Connections:
- IC12 pad 4: /5V -> /5V_B
- IC12 pad 5: /5V -> /5V_B
- IC13 pad 2: /PSU/-3V3_EN_n -> GND
- JP1 pad 1: /3V3_RASP_OUT -> /PSU/5V_A_EN
- JP1 pad 2: Net-(D3-K) -> GND
- JP2 pad 1: /3V3_RASP_OUT -> /PSU/6V_EN
- JP2 pad 2: Net-(D4-K) -> GND
- JP3 pad 1: /3V3_RASP_OUT -> /PSU/5V_B_EN
- JP3 pad 2: Net-(D9-K) -> GND
- JP4 pad 1: /3V3_RASP_OUT -> /PSU/12V_EN
- JP4 pad 2: Net-(D10-K) -> GND
- U1 pad 12: /12V_EN_SW_n -> unconnected-(U1-GPIO9-Pad12)
- U1 pad 19: /6V_EN_SW_n -> unconnected-(U1-GPIO14-Pad19)
- U1 pad 20: /5V_A_EN_SW_n -> unconnected-(U1-GPIO15-Pad20)_0
- U1 pad 24: /5V_B_EN_SW_n -> unconnected-(U1-GPIO18-Pad24)_0
- U1 pad 25: /3V3_A_EN_SW_n -> unconnected-(U1-GPIO19-Pad25)_0
- U1 pad 26: /3V3_B_EN_SW_n -> unconnected-(U1-GPIO20-Pad26)
- U1 pad 27: /-3V3_EN_SW -> unconnected-(U1-GPIO21-Pad27)
Routing:
- net /6V: track 0.00 -> 597.5 mm, vias 0 -> 3
- net /24V: track 0.00 -> 539.0 mm, vias 0 -> 2
- net /3V3_A: track 0.00 -> 526.0 mm, vias 0 -> 13
- net /12V: track 0.00 -> 516.1 mm
- net /5V_B: track 0.00 -> 462.6 mm, vias 0 -> 10
- net /-3V3: track 0.00 -> 346.9 mm, vias 0 -> 10
- net /3V3_B: track 0.00 -> 312.7 mm, vias 0 -> 4
- net /SPI0_SCK: track 0.00 -> 285.6 mm
- net /SPI0_MOSI: track 0.00 -> 285.3 mm
- net /5V_A: track 0.00 -> 274.5 mm, vias 0 -> 2
- net /YIG_CS_n: track 0.00 -> 258.9 mm, vias 0 -> 4
- net /PSU/8V: track 0.00 -> 249.1 mm, vias 0 -> 3
- net /APC2_CS_n: track 0.00 -> 220.7 mm, vias 0 -> 4
- net /SPI1_SCK: track 0.00 -> 203.5 mm, vias 0 -> 7
- net /SPI1_MOSI: track 0.00 -> 197.4 mm, vias 0 -> 6
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Other:
- board text added: "-3V3"
- board text added: "-3V3 OUT"
- board text added: "-3V3 PWR"
- board text added: "-6V"
- board text added: "-6V IN"
- board text added: "-6V_INT"
- board text added: "12V"
- board text added: "12V OUT"
- board text added: "12V PWR"
- board text added: "12V_EN"
- board text added: "14V"
- board text added: "14V IN"
- board text added: "14V_INT"
- board text added: "24V IN"
- board text added: "24V OUT"
- board text added: "24V PWR"
- board text added: "3V3_A"
- board text added: "3V3_A OUT"
- board text added: "3V3_A PWR"
- board text added: "3V3_A_EN"
- board text added: "3V3_B"
- board text added: "3V3_B OUT"
- board text added: "3V3_B PWR"
- board text added: "3V3_B_EN"
- board text added: "5V_A"
- board text added: "5V_A OUT"
- board text added: "5V_A PWR"
- board text added: "5V_A_EN"
- board text added: "5V_B"
- board text added: "5V_B OUT"
- board text added: "5V_B PWR"
- board text added: "5V_B_EN"
- board text added: "6V"
- board text added: "6V OUT"
- board text added: "6V PWR"
- board text added: "6V_AUX"
- board text added: "6V_AUX OUT"
- board text added: "6V_EN"
- board text added: "8V"
- board text added: "8V IN"
- board text added: "8V_INT"
- board text added: "OFF"
- board text added: "ON"
- board text added: "UART"
- board text added: "YIG 1"
- board text added: "YIG 2"

Commit message: Generate QPCB production files
Parts:
- added G***: LOGO, LOGO, F.Cu at (292.7, 68.8)
- added G***: LOGO, LOGO, F.Cu at (292.7, 55.8)
- added G***: LOGO, LOGO, F.Cu at (293.2, 80.0)

Commit message: Last commit from loaner
Parts:
- moved MUXOUT_2 0.72 mm to (328.5, 232.0)
- moved MUXOUT_1 0.66 mm to (339.0, 232.0)
Routing:
- net /24V: track 539.0 -> 555.6 mm
