File: hardware/local_oscillator/kicad/LO_daughter/LO_daughter.kicad_sch (KiCad schematic)
At the start: 43 parts, among them J1 Conn_01x09, J2 Conn_01x09, J3 SMA-J-P-H-ST-TH1, U1 ADF5355, U2 EP2W_, U3 NCR2-113+, U4 EP2W_, U5 SMA-J-P-H-ST-TH1, U6 SMA-J-P-H-ST-TH1, j4 SMA-J-P-H-ST-TH1

Commit message: Generate QPCB production files
Parts:
- U1: LCSC (none) -> C514325; Manufacturer_Name (none) -> Analog Devices; Manufacturer_Part_Number (none) -> ADF5355BCPZ; Mouser Part Number (none) -> 584-ADF5355BCPZ; Mouser Price/Stock (none) -> https://www.mouser.it/ProductDetail/Analog-Devices/ADF5355B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
- U2, U4: LCSC (none) -> C3154895; Manufacturer_Name (none) -> Mini-Circuits; Manufacturer_Part_Number (none) -> EP2W+; Mouser Part Number (none) -> 139-EP2W; Mouser Price/Stock (none) -> https://www.mouser.it/ProductDetail/Mini-Circuits/EP2W%2b?q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
- U3: LCSC (none) -> C3304869; Manufacturer_Name (none) -> Mini-Circuits; Manufacturer_Part_Number (none) -> NCR2-113+; Mouser Part Number (none) -> 139-NCR2-113; Mouser Price/Stock (none) -> https://www.mouser.it/ProductDetail/Mini-Circuits/NCR2-113%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
