File: hardware/amplifier/kicad/amplifier.kicad_pcb (KiCad board)
At the start: 2 copper layers, 35.6 x 26.2 mm, 16 parts, among them J1 SMA-J-P-H-ST-TH1, J2 SMA-J-P-H-ST-TH1, J3 Conn_01x04, J4 Conn_01x04, U1 TSY-83LN+

Commit message: PMA3-83LN+ amplifier
Parts:
- removed C5: 0.4p, Capacitor_SMD:C_0402_1005Metric_Pad0.74x0.62mm_HandSolder
- removed C6: 0.3p, Capacitor_SMD:C_0402_1005Metric_Pad0.74x0.62mm_HandSolder
- removed L3: 2n, Capacitor_SMD:C_0402_1005Metric_Pad0.74x0.62mm_HandSolder
- removed R1: 0, Capacitor_SMD:C_0402_1005Metric_Pad0.74x0.62mm_HandSolder
- removed R2: RADJ, Capacitor_SMD:C_0402_1005Metric_Pad0.74x0.62mm_HandSolder
- L1: renamed from L2; value 22n -> 18n; footprint Capacitor_SMD:C_0402_1005Metric_Pad0.74x0.62mm_HandSolder -> Inductor_SMD:L_0402_1005Metric
- L2: renamed from L1; value L -> 39n; footprint Capacitor_SMD:C_0402_1005Metric_Pad0.74x0.62mm_HandSolder -> Inductor_SMD:L_0402_1005Metric
- U1: value TSY-83LN+ -> PMA3-83LN+; footprint Package_DFN_QFN:QFN-12-1EP_3x3mm_P0.51mm_EP1.45x1.45mm -> footprints:QFN51P300X300X89-13N
- moved L1 3.14 mm to (141.6, 104.3)
- moved L2 1.78 mm to (148.1, 103.3)
- moved C3 1.00 mm to (139.6, 103.8)
- moved C4 1.00 mm to (150.7, 103.8)
Connections:
- C3 pad 2: Net-(U1-RF-IN) -> Net-(C3-Pad2)
- C4 pad 1: Net-(U1-RF-OUT) -> Net-(C4-Pad1)
- L1 pad 1: /RF_IN -> Net-(C3-Pad2)
- L2 pad 2: Net-(U1-VDD) -> Net-(C4-Pad1)
- U1 pad 11: Net-(U1-VEN) -> unconnected-(U1-Pad11)
- U1 pad 12: Net-(U1-IADJ) -> unconnected-(U1-Pad12)
- U1 pad 2: Net-(U1-RF-IN) -> Net-(C3-Pad2)
- U1 pad 8: Net-(U1-RF-OUT) -> Net-(C4-Pad1)
- U1 pad 9: Net-(U1-VDD) -> GND
Routing:
- net GND: track 3.30 -> 13.4 mm, vias 61 -> 0
- net Net-(U1-VEN): track 5.56 -> 0.00 mm
- net unconnected-(U1-Pad12): track 0.00 -> 4.01 mm
- net Net-(C3-Pad2): track 0.00 -> 3.83 mm
- net Net-(C4-Pad1): track 0.00 -> 3.80 mm
- net unconnected-(U1-Pad11): track 0.00 -> 3.79 mm
- net Net-(U1-IADJ): track 3.41 -> 0.00 mm
- net Net-(U1-RF-OUT): track 2.54 -> 0.00 mm
- net Net-(U1-RF-IN): track 2.54 -> 0.00 mm
- net Net-(U1-VDD): track 2.10 -> 0.00 mm
- net /VDD: track 16.0 -> 17.0 mm
- net /RF_OUT: track 6.93 -> 5.93 mm
- net /RF_IN: track 6.93 -> 5.93 mm
